File: kicad/memento-mori.kicad_sch (KiCad schematic)
At the start: 9 parts, among them SW1 SW_SPST, SW2 RotaryEncoder, U1 NodeMCU1.0(ESP-12E)

Commit message: fix schematic
Connections:
- net at Brd1.3 (SCL): now also U1.29 (D1(GPIO5)); no longer U1.26 (D4(GPIO2))
- net at Brd1.4 (SDA): now also U1.28 (D2(GPIO4)); no longer U1.27 (D3(GPIO0))
Changed lines of the file:
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@@
   )
   (no_connect (at 133.35 77.47))
+  (no_connect (at 133.35 85.09))
   (no_connect (at 92.71 82.55))
+  (no_connect (at 133.35 87.63))
   (no_connect (at 92.71 95.25))
-  (no_connect (at 133.35 80.01))
   (no_connect (at 92.71 107.95))
   (no_connect (at 92.71 80.01))
@@
   (no_connect (at 92.71 92.71))
   (no_connect (at 92.71 85.09))
-  (no_connect (at 133.35 82.55))
   (no_connect (at 92.71 90.17))
   (no_connect (at 92.71 97.79))
@@
     (stroke (width 0) (type default) (color 0 0 0 0))
   )
-  (wire (pts (xy 137.16 85.09) (xy 137.16 76.2))
-    (stroke (width 0) (type default) (color 0 0 0 0))
-  )
   (wire (pts (xy 166.37 81.28) (xy 142.24 81.28))
     (stroke (width 0) (type default) (color 0 0 0 0))
@@
     (stroke (width 0) (type default) (color 0 0 0 0))
   )
-  (wire (pts (xy 133.35 87.63) (xy 139.7 87.63))
-    (stroke (width 0) (type default) (color 0 0 0 0))
-  )
   (wire (pts (xy 88.9 110.49) (xy 88.9 100.33))
     (stroke (width 0) (type default) (color 0 0 0 0))
   )
   (wire (pts (xy 163.83 116.84) (xy 179.07 116.84))
-    (stroke (width 0) (type default) (color 0 0 0 0))
-  )
-  (wire (pts (xy 133.35 85.09) (xy 137.16 85.09))
     (stroke (width 0) (type default) (color 0 0 0 0))
   )
@@
     (stroke (width 0) (type default) (color 0 0 0 0))
   )
-  (wire (pts (xy 139.7 78.74) (xy 166.37 78.74))
+  (wire (pts (xy 156.21 110.49) (xy 156.21 116.84))
     (stroke (width 0) (type default) (color 0 0 0 0))
   )
-  (wire (pts (xy 156.21 110.49) (xy 156.21 116.84))
+  (wire (pts (xy 139.7 80.01) (xy 139.7 78.74))
     (stroke (width 0) (type default) (color 0 0 0 0))
   )
@@
   )
   (wire (pts (xy 163.83 106.68) (xy 163.83 116.84))
+    (stroke (width 0) (type default) (color 0 0 0 0))
+  )
+  (wire (pts (xy 139.7 78.74) (xy 166.37 78.74))
     (stroke (width 0) (type default) (color 0 0 0 0))
   )
@@
     (stroke (width 0) (type default) (color 0 0 0 0))
   )
+  (wire (pts (xy 137.16 82.55) (xy 137.16 76.2))
+    (stroke (width 0) (type default) (color 0 0 0 0))
+  )
   (wire (pts (xy 133.35 92.71) (xy 144.78 92.71))
     (stroke (width 0) (type default) (color 0 0 0 0))
@@
     (stroke (width 0) (type default) (color 0 0 0 0))
   )
-  (wire (pts (xy 139.7 87.63) (xy 139.7 78.74))
+  (wire (pts (xy 133.35 82.55) (xy 137.16 82.55))
     (stroke (width 0) (type default) (color 0 0 0 0))
   )
@@
     (stroke (width 0) (type default) (color 0 0 0 0))
   )
+  (wire (pts (xy 133.35 80.01) (xy 139.7 80.01))
+    (stroke (width 0) (type default) (color 0 0 0 0))
+  )
